File: kicad/kb-tester-shift30.kicad_sch (KiCad schematic)
At the start: 65 parts, among them J1 Conn_01x12_Pin, J2 Conn_01x05_Socket, J3 8-1437565-1, SW1 PG1350, SW10 PG1350, SW11 PG1350, SW12 PG1350, SW13 PG1350, SW14 PG1350, SW15 PG1350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

Commit message: Add production
Parts:
- D1, D10, D11, D12, D13, D14, D15, D16, D17, D18, D19, D2, D20, D21, D22, D23, D24, D25, D26, D27, D28, D29, D3, D30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: Comment (none) -> 1N4148W; JLCPCB Part # (none) -> C81598
- J3: now not fitted
- U2: Comment (none) -> SOIC-16:74HC595D,118; JLCPCB Part # (none) -> C5947
