File: kicad/kb-devboard.kicad_pcb (KiCad board)
At the start: 2 copper layers, 109.7 x 91.8 mm, 122 parts, among them J1 Conn_01x14_Pin, SW1 PG1350, SW10 PG1350, SW11 PG1350, SW12 PG1350, SW13 PG1350, SW14 PG1350, SW15 PG1350, SW16 PG1350, SW17 PG1350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

Commit message: Update to rev b
Other:
- board text added: "REV B 4/24"
- board text removed: "REV.A 4/24"
Changed lines of the file:
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@@
 		(layer "Edge.Cuts")
 	)
-	(gr_text "REV.A 4/24"
+	(gr_text "REV B 4/24"
 		(at 123.4 48.7 0)
 		(layer "B.SilkS")
