File: kicad/kb-devboard.kicad_sch (KiCad schematic)
At the start: 121 parts, among them J1 Conn_01x14_Pin, SW1 PG1350, SW10 PG1350, SW11 PG1350, SW12 PG1350, SW13 PG1350, SW14 PG1350, SW15 PG1350, SW16 PG1350, SW17 PG1350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

Commit message: Update to rev b
Other:
- moved on the sheet: D1, D10, D11, D12, D13, D14, D15, D16, D17, D18, D19, D2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
